File: MCU.kicad_sch (KiCad schematic)
At the start: 17 parts, among them U3 STM32L476RGTx, Y1 Crystal

Commit message: Add ChipSat inhibit
Connections:
- net INHIBIT: now reaches U3.50 (PA15)
- no-connect marks 16 -> 15
Changed lines of the file:
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@@
   (no_connect (at 224.79 146.05))
   (no_connect (at 224.79 113.03))
-  (no_connect (at 224.79 128.27))
   (no_connect (at 189.23 168.91))
   (no_connect (at 189.23 143.51))
@@
     (effects (font (size 1.524 1.524)) (justify right))
   )
+  (hierarchical_label "INHIBIT" (shape input) (at 224.79 128.27 0) (fields_autoplaced)
+    (effects (font (size 1.27 1.27)) (justify left))
+  )
   (hierarchical_label "CAN_STB" (shape input) (at 224.79 138.43 0) (fields_autoplaced)

Commit message: Update some part numbers
Parts:
- C9: Part Number GRM188R60J475KE19D -> GRT188R60J475KE01D
- D2: Part Number (none) -> LTST-C190KFKT
- D3: Part Number (none) -> LTST-C190KRKT
- R10: MPN (none) -> RE0603BRE0710KL; Part Number (none) -> RE0603BRE0710KL
- R11: Part Number (none) -> RMCF0603FT47K0
- R8, R9: MPN (none) -> RE0603BRE0710KL
- Y1: Part Number (none) -> ECS-80-18-5PX-CKM-TR
Changed lines of the file:
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@@
       (effects (font (size 1.27 1.27)) hide)
     )
-    (property "Part Number" "GRM188R60J475KE19D" (at 229.87 74.93 0)
+    (property "Part Number" "GRT188R60J475KE01D" (at 229.87 74.93 0)
       (effects (font (size 1.27 1.27)) hide)
     )
@@
       (effects (font (size 1.27 1.27)) hide)
     )
+    (property "Part Number" "ECS-80-18-5PX-CKM-TR" (at 170.18 121.92 0)
+      (effects (font (size 1.27 1.27)) hide)
+    )
     (pin "1")
     (pin "2")
@@
       (effects (font (size 1.27 1.27)) hide)
     )
+    (property "Part Number" "RMCF0603FT47K0" (at 278.13 142.24 0)
+      (effects (font (size 1.27 1.27)) hide)
+    )
     (pin "1")
     (pin "2")
@@
       (effects (font (size 1.27 1.27)) hide)
     )
+    (property "Part Number" "LTST-C190KFKT" (at 288.29 127 0)
+      (effects (font (size 1.27 1.27)) hide)
+    )
     (pin "1")
     (pin "2")
@@
       (effects (font (size 1.27 1.27)) hide)
     )
+    (property "MPN" "RE0603BRE0710KL" (at 186.69 83.82 0)
+      (effects (font (size 1.27 1.27)) hide)
+    )
     (pin "1")
     (pin "2")
@@
       (effects (font (size 1.27 1.27)) hide)
     )
+    (property "Part Number" "LTST-C190KRKT" (at 288.29 142.24 0)
+      (effects (font (size 1.27 1.27)) hide)
+    )
     (pin "1")
     (pin "2")
@@
       (effects (font (size 1.27 1.27)) hide)
     )
+    (property "MPN" "RE0603BRE0710KL" (at 185.42 99.06 0)
+      (effects (font (size 1.27 1.27)) hide)
+    )
     (pin "1")
     (pin "2")
@@
       (effects (font (size 1.27 1.27)) hide)
     )
+    (property "MPN" "RE0603BRE0710KL" (at 278.13 127 0)
+      (effects (font (size 1.27 1.27)) hide)
+    )
+    (property "Part Number" "RE0603BRE0710KL" (at 278.13 127 0)
+      (effects (font (size 1.27 1.27)) hide)
+    )
