File: connectors.kicad_sch (KiCad schematic)
At the start: 12 parts, among them J2 MTQZ, J6 MTQZ

Commit message: Update some part numbers
Parts:
- J6: Part Number (none) -> SQT-102-03-F-S
- R4, R5, R6, R7: Part Number (none) -> ERA-6AEB5902V
Changed lines of the file:
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@@
+      (effects (font (size 1.27 1.27)) hide)
+    )
+    (property "Part Number" "ERA-6AEB5902V" (at 116.84 67.31 0)
       (effects (font (size 1.27 1.27)) hide)
     )
@@
     (property "MANUFACTURER" "SAMTEC" (at 175.26 76.2 0)
       (effects (font (size 1.27 1.27)) (justify bottom) hide)
+    )
+    (property "Part Number" "SQT-102-03-F-S" (at 175.26 76.2 0)
+      (effects (font (size 1.27 1.27)) hide)
     )
     (pin "01")
@@
     )
     (property "MPN" "ERA-6AEB5902V" (at 116.84 146.05 0)
+      (effects (font (size 1.27 1.27)) hide)
+    )
+    (property "Part Number" "ERA-6AEB5902V" (at 116.84 146.05 0)
       (effects (font (size 1.27 1.27)) hide)
     )
@@
       (effects (font (size 1.27 1.27)) hide)
     )
+    (property "Part Number" "ERA-6AEB5902V" (at 116.84 93.98 0)
+      (effects (font (size 1.27 1.27)) hide)
+    )
     (pin "1")
     (pin "2")
@@
       (effects (font (size 1.27 1.27)) hide)
     )
+    (property "Part Number" "ERA-6AEB5902V" (at 116.84 119.38 0)
+      (effects (font (size 1.27 1.27)) hide)
+    )
