File: NEW_PCB_ADCS.kicad_pcb (KiCad board)
At the start: 2 copper layers, 42 x 42 mm, 80 parts, among them IC1 DRV8212DSGR, IC2 DRV8212DSGR, IC3 DRV8212DSGR, J1 SWD, J2 MTQZ, J6 MTQZ, J7 Micro_SD_Card_Det_Hirose_DM3AT, J8 PQ9-Connector, U1 AD8603, U2 47K, U3 STM32L476RGTx, U4 TCAN334, U5 LIS3MDL, U6 BNO055, Y1 Crystal

Commit message: Add fiducials
Parts:
- added REF**: Fiducial_3mm_Mask5mm, POQUITO_Panel_Library:Fiducial_3mm_Mask5mm, F.Cu at (179.2, 95.1)
- added REF**: Fiducial_3mm_Mask5mm, POQUITO_Panel_Library:Fiducial_3mm_Mask5mm, F.Cu at (209.2, 95.1)
Changed lines of the file:
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@@
     )
   )
+  (footprint "POQUITO_Panel_Library:Fiducial_3mm_Mask5mm" (layer "F.Cu")
+    (at 179.2 95.1)
+    (descr "Circular Fiducial, 1.5mm bare copper, 4.5mm soldermask opening")
+    (tags "fiducial")
+    (attr smd)
+    (fp_text reference "REF**" (at 0 -3.175) (layer "F.SilkS")
+        (effects (font (size 1 1) (thickness 0.15)))
+    )
+    (fp_text value "Fiducial_3mm_Mask5mm" (at 0 3.175) (layer "F.Fab")
+        (effects (font (size 1 1) (thickness 0.15)))
+    )
+    (fp_text user "${REFERENCE}" (at 0 0) (layer "F.Fab")
+        (effects (font (size 0.4 0.4) (thickness 0.06)))
+    )
+    (fp_circle (center 0 0) (end 2.5 0)
+      (stroke (width 0.05) (type solid)) (fill none) (layer "F.CrtYd"))
+    (fp_circle (center 0 0) (end 2.5 0)
+      (stroke (width 0.1) (type solid)) (fill none) (layer "F.Fab"))
+    (pad "" smd circle (at 0 0) (size 3 3) (layers "F.Cu" "F.Mask")
+      (solder_mask_margin 1) (clearance 1))
+  )
   (footprint "Capacitor_SMD:C_0603_1608Metric" (layer "F.Cu")
     (at 203.962 70.203 90)
@@
     )
   )
+  (footprint "POQUITO_Panel_Library:Fiducial_3mm_Mask5mm" (layer "F.Cu")
+    (at 209.2 95.1)
+    (descr "Circular Fiducial, 1.5mm bare copper, 4.5mm soldermask opening")
+    (tags "fiducial")
+    (attr smd)
+    (fp_text reference "REF**" (at 0 -3.175) (layer "F.SilkS")
+        (effects (font (size 1 1) (thickness 0.15)))
+    )
+    (fp_text value "Fiducial_3mm_Mask5mm" (at 0 3.175) (layer "F.Fab")
+        (effects (font (size 1 1) (thickness 0.15)))
+    )
+    (fp_text user "${REFERENCE}" (at 0 0) (layer "F.Fab")
+        (effects (font (size 0.4 0.4) (thickness 0.06)))
+    )
+    (fp_circle (center 0 0) (end 2.5 0)
+      (stroke (width 0.05) (type solid)) (fill none) (layer "F.CrtYd"))
+    (fp_circle (center 0 0) (end 2.5 0)
+      (stroke (width 0.1) (type solid)) (fill none) (layer "F.Fab"))
+    (pad "" smd circle (at 0 0) (size 3 3) (layers "F.Cu" "F.Mask")
+      (solder_mask_margin 1) (clearance 1))
+  )
   (footprint "Package_QFP:LQFP-64_10x10mm_P0.5mm" (layer "F.Cu")
     (at 191.806 65.445 -90)
@@
     (effects (font (size 0.7 0.7) (thickness 0.12) bold) (justify bottom))
   )
+  (dimension (type orthogonal) (layer "Cmts.User")
+    (pts (xy 176.1872 90.5942) (xy 177.8 95.1))
+    (height 50.009255)
+    (orientation 1)
+    (gr_text "4.5058 mm" (at 225.046455 92.8471 90) (layer "Cmts.User")
+      (effects (font (size 1 1) (thickness 0.15)))
+    )
+    (format (prefix "") (suffix "") (units 3) (units_format 1) (precision 4))
+    (style (thickness 0.15) (arrow_length 1.27) (text_position_mode 0) (extension_height 0.58642) (extension_offset 0.5) keep_text_aligned)
+  )
+  (dimension (type orthogonal) (layer "Cmts.User")
+    (pts (xy 173.1872 85.5942) (xy 194.19 85.33))
+    (height 25.0458)
+    (orientation 0)
+    (gr_text "21.0028 mm" (at 183.6886 109.49) (layer "Cmts.User")
+      (effects (font (size 1 1) (thickness 0.15)))
+    )
+    (format (prefix "") (suffix "") (units 3) (units_format 1) (precision 4))
+    (style (thickness 0.15) (arrow_length 1.27) (text_position_mode 0) (extension_height 0.58642) (extension_offset 0.5) keep_text_aligned)
+  )
+  (dimension (type orthogonal) (layer "Cmts.User")
+    (pts (xy 194.2 102.4) (xy 179.2 102.1))
+    (height 4.323628)
+    (orientation 0)
+    (gr_text "15.0000 mm" (at 186.7 105.573628) (layer "Cmts.User")
+      (effects (font (size 1 1) (thickness 0.15)))
+    )
+    (format (prefix "") (suffix "") (units 3) (units_format 1) (precision 4))
+    (style (thickness 0.15) (arrow_length 1.27) (text_position_mode 0) (extension_height 0.58642) (extension_offset 0.5) keep_text_aligned)
+  )
+  (dimension (type orthogonal) (layer "Cmts.User")
+    (pts (xy 194.2 102.4) (xy 209.2 102.4))
+    (height 4.3)
+    (orientation 0)
+    (gr_text "15.0000 mm" (at 201.7 105.55) (layer "Cmts.User")
+      (effects (font (size 1 1) (thickness 0.15)))
+    )
+    (format (prefix "") (suffix "") (units 3) (units_format 1) (precision 4))
+    (style (thickness 0.15) (arrow_length 1.27) (text_position_mode 0) (extension_height 0.58642) (extension_offset 0.5) keep_text_aligned)
+  )
   (segment (start 194.056 61.359955) (end 194.056 59.77) (width 0.25) (layer "F.Cu") (net 1))

Commit message: Fix footprints, brought to you by Spyros
Parts:
- U2: footprint lsf-kicad-lib:EXBD -> LocalLibrary:EXBD
- Y1: footprint Crystal:Crystal_SMD_ECS_CSM3X-2Pin_7.6x4.1mm -> LocalLibrary:ECS-080-18-23G-JGN-TR
Routing:
- net Net-(U3-PH0): track 18.2 -> 18.7 mm
